File: pmod-uext.kicad_sch (KiCad schematic)
At the start: 9 parts, among them J1 61301221021, J2 61201021621, SW1 219-2MST, U1 TMUX1309PWR, U2 TMUX1309PWR, U3 TMUX1309PWR, U4 TMUX1309PWR

Commit message: change project metas
- rename files with more accurate names
- remove unnecessary files
- improve documents, also reflect structural changes
Parts:
- U1, U2, U3, U4: symbol PMOD-UEXT:TMUX1309 -> pmod-uext:TMUX1309
Changed lines of the file:
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@@
 		)
 		(instances
-			(project "PMOD-UEXT"
+			(project "pmod-uext"
 				(path "/382daf84-bf7b-44ad-8559-ab4145e50afa"
 					(reference "#PWR08")
@@
 		)
 		(instances
-			(project "PMOD-UEXT"
+			(project "pmod-uext"
 				(path "/382daf84-bf7b-44ad-8559-ab4145e50afa"
 					(reference "#PWR011")
@@
 		)
 		(instances
-			(project "PMOD-UEXT"
+			(project "pmod-uext"
 				(path "/382daf84-bf7b-44ad-8559-ab4145e50afa"
 					(reference "#PWR015")
@@
 		)
 		(instances
-			(project "PMOD-UEXT"
+			(project "pmod-uext"
 				(path "/382daf84-bf7b-44ad-8559-ab4145e50afa"
 					(reference "#PWR017")
@@
 	)
 	(symbol
-		(lib_id "PMOD-UEXT:TMUX1309")
+		(lib_id "pmod-uext:TMUX1309")
 		(at 165.1 119.38 0)
 		(unit 1)
@@
 	)
 	(symbol
-		(lib_id "PMOD-UEXT:TMUX1309")
+		(lib_id "pmod-uext:TMUX1309")
 		(at 49.53 119.38 0)
 		(unit 1)
@@
 		)
 		(instances
-			(project "PMOD-UEXT"
+			(project "pmod-uext"
 				(path "/382daf84-bf7b-44ad-8559-ab4145e50afa"
 					(reference "#PWR016")
@@
 		)
 		(instances
-			(project "PMOD-UEXT"
+			(project "pmod-uext"
 				(path "/382daf84-bf7b-44ad-8559-ab4145e50afa"
 					(reference "#PWR020")
@@
 		)
 		(instances
-			(project "PMOD-UEXT"
+			(project "pmod-uext"
 				(path "/382daf84-bf7b-44ad-8559-ab4145e50afa"
 					(reference "#PWR010")
@@
 		)
 		(instances
-			(project "PMOD-UEXT"
+			(project "pmod-uext"
 				(path "/382daf84-bf7b-44ad-8559-ab4145e50afa"
 					(reference "#PWR021")
@@
 	)
 	(symbol
-		(lib_id "PMOD-UEXT:TMUX1309")
+		(lib_id "pmod-uext:TMUX1309")
 		(at 107.95 119.38 0)
 		(unit 1)
@@
 		)
 		(instances
-			(project "PMOD-UEXT"
+			(project "pmod-uext"
 				(path "/382daf84-bf7b-44ad-8559-ab4145e50afa"
 					(reference "#PWR022")
@@
 	)
 	(symbol
-		(lib_id "PMOD-UEXT:TMUX1309")
+		(lib_id "pmod-uext:TMUX1309")
 		(at 223.52 119.38 0)
 		(unit 1)
